File: Moka.sch (KiCad schematic (older format))
At the start: 66 parts, among them J1 CONN_02X03, J10 CONN_01X05, J2 GS2, J3 GS2, J4 GS2, J5 GS2, J6 GS2, J7 CONN_01X05, J8 CONN_01X05, J9 CONN_01X05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

Commit message: Design ok, first prototype batch ordered.
Parts:
- added logo1: Moka, Logos:Moka_20mm, symbol Logo
- added logo2: le labo, Logos:Logo_labo_20mm, symbol Logo
Changed lines of the file:
@@
 LIBS:switches
 LIBS:Holes_Fids
+LIBS:Logos
 LIBS:Tuile-cache
 EELAYER 25 0
@@
 	8050 3100 8100 3100
 Connection ~ 8100 3100
+$Comp
+L Logo logo1
+U 1 1 594E8880
+P 6550 6950
+F 0 "logo1" H 6550 7050 60  0000 C CNN
+F 1 "Moka" H 6550 6850 60  0000 C CNN
+F 2 "Logos:Moka_20mm" H 6550 6950 60  0001 C CNN
+F 3 "" H 6550 6950 60  0001 C CNN
+	1    6550 6950
+	1    0    0    -1
+$EndComp
+$Comp
+L Logo logo2
+U 1 1 594E93C5
+P 6550 7300
+F 0 "logo2" H 6550 7400 60  0000 C CNN
+F 1 "le labo" H 6550 7200 60  0000 C CNN
+F 2 "Logos:Logo_labo_20mm" H 6550 7300 60  0001 C CNN
+F 3 "" H 6550 7300 60  0001 C CNN
+	1    6550 7300
+	1    0    0    -1
+$EndComp
 $EndSCHEMATC

Commit message: v0.95 ready for fabrication.
Parts:
- removed D1, D10, D11, D12, D13, D14, D15, D16, D2, D3, D4, D5, D6, D7, D8, D9: Led_3535_addr, Display_perso:SK6812-mini, symbol Led_3535_addr
- removed J1: CONN_02X03, Conn_perso:Pin_Header_Straight_2x03_Pitch2.54mm_SMD, symbol CONN_02X03
- added D1: D, Diodes_SMD:D_0603, symbol D
- added D10, D11, D12, D13, D14, D15, D16, D17, D2, D3, D4, D5, D6, D7, D8, D9: SK6812_MINI, Display_perso:SK6812-mini, symbol SK6812_MINI
- added J1: Conn_02x03_Odd_Even, Connectors_perso:Pin_Header_Straight_2x03_Pitch2.54mm_SMD, symbol Conn_02x03_Odd_Even
- J10, J7, J8, J9: footprint Conn_perso:Connecteur_1x5_SMD -> Connectors_perso:Connecteur_1x5_SMD; symbol CONN_01X05 -> Conn_01x05
- SW1, SW10, SW11, SW12, SW13, SW14, SW15, SW16, SW2, SW3, SW4, SW5, SW6, SW7, SW8, SW9: footprint Switches_perso:Pad_30 -> switches_perso:Pad_30
- logo1: footprint Logos:Moka_20mm -> logos:Moka_25mm
- logo2: footprint Logos:Logo_labo_20mm -> logos:Le_labo_20mm
Connections:
- net labels added: BCH1, BCH2, BCH3, BCH4, BREAD1, BREAD2, BREAD3, BREAD4
- net labels removed: BIN1, BIN2, BIN3, BIN4, BOUT1, BOUT2, BOUT3, BOUT4
- wire segments 193 -> 199
Other:
- moved on the sheet: R1, R2, R3

Commit message: Modified diode footprint on INT.
Parts:
- D1: footprint Diodes_SMD:D_0603 -> Diodes_SMD:D_SOD-123
Changed lines of the file:
@@
 EESchema Schematic File Version 2
 LIBS:Moka-rescue
-LIBS:Tuile-rescue
 LIBS:power
 LIBS:device
@@
 F 0 "D1" H 4550 1500 50  0000 C CNN
 F 1 "D" H 4550 1300 50  0000 C CNN
-F 2 "Diodes_SMD:D_0603" H 4550 1400 50  0001 C CNN
+F 2 "Diodes_SMD:D_SOD-123" H 4550 1400 50  0001 C CNN
 F 3 "" H 4550 1400 50  0001 C CNN
 	1    4550 1400
